File: keycopy.brd (EAGLE design)
At the start: 102.2 x 38.1 mm, 85 parts

Commit message: b002
Parts:
- C1*: value 2n -> 2n2
- C1B*: value 2n -> (none)
- C8: value 150n -> 100n
- C8B: value 150n -> 47n
- DISP: value TUXGR_16X2_R21 -> QC1602A V2.0
- L1: value 820mkhn -> 777
- R: value 1k -> 10k
- TEST_PIN: value (none) -> +30V
Changed lines of the file:
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@@
 <attribute name="VALUE" x="63.8175" y="34.29" size="1.27" layer="27" rot="R180"/>
 </element>
-<element name="C1*" library="keycopy" package="C025-030X050" value="2n" x="72.7075" y="3.4925" smashed="yes" rot="R270">
+<element name="C1*" library="keycopy" package="C025-030X050" value="2n2" x="72.7075" y="3.4925" smashed="yes" rot="R270">
 <attribute name="NAME" x="74.549" y="6.604" size="1.27" layer="25" ratio="10"/>
 <attribute name="VALUE" x="69.9135" y="5.7785" size="1.27" layer="27" ratio="10" rot="R270"/>
@@
 <attribute name="VALUE" x="39.37" y="2.54" size="1.27" layer="28" rot="MR0"/>
 </element>
-<element name="C8" library="keycopy" package="C025-030X050" value="150n" x="35.56" y="3.4925" smashed="yes" rot="R270">
+<element name="C8" library="keycopy" package="C025-030X050" value="100n" x="35.56" y="3.4925" smashed="yes" rot="R270">
 <attribute name="NAME" x="34.8615" y="6.2865" size="1.27" layer="25" ratio="10"/>
 <attribute name="VALUE" x="32.766" y="5.7785" size="1.27" layer="27" ratio="10" rot="R270"/>
 </element>
-<element name="TEST_PIN" library="keycopy" package="1X01" value="" x="63.8175" y="6.6675" smashed="yes" rot="R90">
+<element name="TEST_PIN" library="keycopy" package="1X01" value="+30V" x="63.8175" y="6.6675" smashed="yes" rot="R90">
 <attribute name="NAME" x="63.5762" y="8.4963" size="1.27" layer="25" ratio="10" rot="R90"/>
 <attribute name="VALUE" x="66.9925" y="5.3975" size="1.27" layer="27" rot="R90"/>
@@
 <element name="U$7" library="HWProgUSB" package="PROGRAMMER_KEY" value="PROGRAMMER_5.08" x="98.7425" y="23.8125" smashed="yes" rot="R90"/>
 <element name="U$8" library="HWProgUSB" package="PROGRAMMER_KEY" value="PROGRAMMER_5.08" x="86.0425" y="23.8125" smashed="yes" rot="R90"/>
-<element name="DISP" library="keycopy" package="TUXGR_16X2_1" value="TUXGR_16X2_R21" x="40.5638" y="18.4912" smashed="yes">
+<element name="DISP" library="keycopy" package="TUXGR_16X2_1" value="QC1602A V2.0" x="40.5638" y="18.4912" smashed="yes">
 <attribute name="NAME" x="2.4638" y="36.9062" size="1.27" layer="25"/>
 <attribute name="VALUE" x="41.1988" y="36.9062" size="1.27" layer="27"/>
 </element>
-<element name="L1" library="keycopy" package="0207/2V" value="820mkhn" x="78.74" y="9.2075" smashed="yes" rot="R270">
+<element name="L1" library="keycopy" package="0207/2V" value="777" x="78.74" y="9.2075" smashed="yes" rot="R270">
 <attribute name="NAME" x="78.3717" y="12.1285" size="1.27" layer="25" ratio="10"/>
 <attribute name="VALUE" x="76.5048" y="9.2583" size="1.27" layer="27" ratio="10" rot="R270"/>
 </element>
-<element name="C8B" library="keycopy" package="C025-030X050" value="150n" x="32.385" y="3.4925" smashed="yes" rot="R270">
+<element name="C8B" library="keycopy" package="C025-030X050" value="47n" x="32.385" y="3.4925" smashed="yes" rot="R270">
 <attribute name="NAME" x="31.0515" y="6.35" size="1.27" layer="25" ratio="10"/>
 <attribute name="VALUE" x="29.337" y="5.7785" size="1.27" layer="27" ratio="10" rot="R270"/>
@@
 <attribute name="VALUE" x="66.675" y="12.7" size="1.27" layer="28" rot="MR0"/>
 </element>
-<element name="C1B*" library="keycopy" package="C025-030X050" value="2n" x="69.5325" y="3.4925" smashed="yes" rot="R270">
+<element name="C1B*" library="keycopy" package="C025-030X050" value="" x="69.5325" y="3.4925" smashed="yes" rot="R270">
 <attribute name="NAME" x="74.2315" y="5.08" size="1.27" layer="25" ratio="10"/>
 <attribute name="VALUE" x="66.4845" y="5.7785" size="1.27" layer="27" ratio="10" rot="R270"/>
@@
 </element>
 <element name="R3B" library="keycopy" package="M0805" value="1k5" x="63.1825" y="31.75" rot="MR0"/>
-<element name="R" library="rcl" package="R0805" value="1k" x="53.975" y="26.035" smashed="yes" rot="MR225">
+<element name="R" library="rcl" package="R0805" value="10k" x="53.975" y="26.035" smashed="yes" rot="MR225">
 <attribute name="NAME" x="55.312465625" y="22.282665625" size="1.27" layer="26" ratio="10" rot="MR225"/>
 <attribute name="VALUE" x="54.257915625" y="25.7520875" size="0.02" layer="28" rot="MR225"/>
@@
 <wire x1="35.2425" y1="20.955" x2="36.5125" y2="21.209" width="2.032" layer="16"/>
 <contactref element="R" pad="2"/>
-<wire x1="11.1038" y1="33.9912" x2="33.909" y2="19.8755" width="0" layer="19" extent="16-16"/>
 <wire x1="54.646753125" y1="25.363246875" x2="54.6800625" y2="25.363246875" width="0.3048" layer="16"/>
 <wire x1="54.6800625" y1="25.363246875" x2="55.003790625" y2="25.03951875" width="0.3048" layer="16"/>
+<wire x1="11.1038" y1="33.9912" x2="33.909" y2="19.8755" width="0" layer="19" extent="16-16"/>
 </signal>
 <signal name="N$4">

Commit message: v0.21
Parts:
- C14: value 47n -> 47m
- R3~: value 1k5 -> SMD
- VT1: device transistor-pnp:TO126 -> keycopy:TO126
- moved L3 2.69 mm to (27.0, 19.1)
- moved R11* 1.31 mm to (21.0, 30.2)
- moved C12 0.95 mm to (17.8, 19.1)
- moved VT1 0.95 mm to (30.5, 23.5)
- moved R5 0.64 mm to (41.6, 21.3)
- moved R4* 0.63 mm to (40.3, 24.1)
- moved C13 0.32 mm to (12.4, 14.3)
- moved L2 0.32 mm to (13.3, 25.7)
- moved VD7 0.32 mm to (66.0, 4.45)
- moved VD8 0.32 mm to (20.3, 23.5)
- renumbered R3B to R3~
Connections:
- net V+: now also R4*.2, VT2.E
- net VCC/2: no longer R4*.2, VT2.E
Routing:
- net V+: track 22.9 -> 66.9 mm, vias 0 -> 2
- net VCC/2: track 106.7 -> 101.2 mm
- net B3: track 79.3 -> 77.0 mm
- net B7: track 50.9 -> 52.7 mm
- net VCC: track 96.1 -> 94.4 mm
- net B6: track 51.1 -> 52.8 mm
- net N$4: track 22.4 -> 24.0 mm
- net B5: track 52.1 -> 53.6 mm
- net N$12: track 6.58 -> 5.28 mm
- net N$17: track 4.38 -> 5.65 mm
- net N$24: track 10.4 -> 9.19 mm
- net B4: track 52.0 -> 53.2 mm
- net N$7: track 11.7 -> 12.5 mm
- net A1: track 90.1 -> 90.8 mm
- net N$18: track 1.93 -> 2.56 mm
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
Commit message: v0.22
Routing:
- net GND: track 369.7 -> 370.4 mm, vias 3 -> 4
Changed lines of the file:
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@@
 <setting verticaltext="up"/>
 </settings>
-<grid distance="12.5" unitdist="mil" unit="mil" style="lines" multiple="1" display="yes" altdistance="0.025" altunitdist="inch" altunit="inch"/>
+<grid distance="50" unitdist="mil" unit="mil" style="lines" multiple="1" display="yes" altdistance="0.025" altunitdist="inch" altunit="inch"/>
 <layers>
 <layer number="1" name="Top" color="4" fill="1" visible="yes" active="yes"/>
@@
 </element>
 <element name="C3" library="keycopy" package="CAP-PTH-LARGE" value="3n3" x="21.2725" y="8.09625" smashed="yes" rot="R270">
-<attribute name="NAME" x="22.5425" y="8.85825" size="0.4064" layer="25" rot="R270"/>
+<attribute name="NAME" x="22.89175" y="9.8425" size="1.27" layer="25"/>
 <attribute name="VALUE" x="19.7485" y="9.11225" size="0.4064" layer="27" rot="R270"/>
 </element>
@@
 </element>
 <element name="LED_R" library="keycopy3" package="LED3MM" value="ON" x="91.7575" y="28.8925" smashed="yes">
-<attribute name="NAME" x="92.329" y="31.4325" size="1.27" layer="25" ratio="10" rot="R90"/>
+<attribute name="NAME" x="92.329" y="30.1625" size="1.27" layer="25" ratio="10" rot="R90"/>
 <attribute name="VALUE" x="93.6625" y="27.2415" size="1.27" layer="27" ratio="10"/>
 </element>
@@
 </element>
 <element name="C4" library="keycopy" package="CAP-PTH-LARGE" value="3n3" x="62.865" y="24.765" smashed="yes" rot="R358">
-<attribute name="NAME" x="62.147784375" y="26.06081875" size="0.4064" layer="25" rot="R358"/>
+<attribute name="NAME" x="60.877784375" y="22.25081875" size="1.27" layer="25" rot="R358"/>
 <attribute name="VALUE" x="61.79643125" y="23.277384375" size="0.4064" layer="27" rot="R358"/>
 </element>
@@
 <wire x1="22.6869125" y1="27.1605875" x2="20.6375" y2="28.2575" width="0.4064" layer="16"/>
 <wire x1="20.6375" y1="28.2575" x2="13.97" y2="28.2575" width="0.4064" layer="16"/>
-<wire x1="50.8" y1="23.1775" x2="50.8" y2="34.29" width="0.4064" layer="1"/>
 <wire x1="12.7" y1="29.5275" x2="10.16" y2="29.5275" width="0.4064" layer="16"/>
 <wire x1="10.16" y1="29.5275" x2="8.89" y2="30.21" width="0.4064" layer="16"/>
@@
 </polygon>
 <wire x1="50.8" y1="37.7825" x2="50.8" y2="34.29" width="1.016" layer="16"/>
+<wire x1="50.8" y1="23.1775" x2="51.435" y2="25.7175" width="0.4064" layer="1"/>
+<wire x1="51.435" y1="25.7175" x2="50.4825" y2="27.305" width="0.4064" layer="1"/>
+<wire x1="50.4825" y1="27.305" x2="51.435" y2="28.8925" width="0.4064" layer="1"/>
+<wire x1="51.435" y1="28.8925" x2="50.8" y2="34.29" width="0.4064" layer="1"/>
+<via x="91.7575" y="37.1475" extent="1-16" drill="0.8" diameter="2.3"/>
 <wire x1="8.5725" y1="33.9725" x2="8.5638" y2="33.9912" width="0" layer="19" extent="1-1"/>
 </signal>

Commit message: v0.3
Parts:
- added R4: 1k, rcl:R1206W
- L1: value 777 -> 777uH
- R4*: value 120 -> 20; device rcl:R1206W -> rcl:R0805
- VD2: value 3v9* -> 1v5*
- VT2: value КТ361 -> КТ361Б
- moved R4* 3.00 mm to (38.7, 21.6), turned to 270 degrees
- moved R 0.22 mm to (53.8, 26.2)
Connections:
- new net N$38: R4*.1, R4.2
- net N$17: now also R4.1; no longer R4*.1
Routing:
- net V+: track 66.9 -> 63.7 mm
- net GND: track 370.4 -> 372.1 mm, vias 4 -> 5
- net N$39: track 0.00 -> 1.75 mm
- net N$38: track 0.00 -> 1.59 mm
- net VCC: track 94.4 -> 94.8 mm, vias 0 -> 1

Commit message: v0.33
Parts:
- R21: value 1R -> 0.5R
- moved L1 1.31 mm to (78.4, 10.5)
- moved +3V 0.32 mm to (2.86, 27.6)
Changed lines of the file:
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@@
 <attribute name="MF" value="MICROCHIP" x="21.2725" y="9.525" size="1.778" layer="28" rot="MR0" display="off"/>
 <attribute name="OC_FARNELL" value="9760415" x="21.2725" y="9.525" size="1.778" layer="28" rot="MR0" display="off"/>
-<attribute name="NAME" x="13.0429" y="7.62" size="1.778" layer="26" ratio="10" rot="MR90"/>
+<attribute name="NAME" x="14.605" y="7.9629" size="1.778" layer="26" ratio="10" rot="MR0"/>
 <attribute name="VALUE" x="13.3604" y="5.715" size="1.778" layer="28" ratio="10" rot="MR90"/>
 </element>
@@
 <attribute name="VALUE" x="5.9055" y="27.686" size="1.27" layer="28" rot="MR180"/>
 </element>
-<element name="R21" library="resistor" package="R0805" value="1R" x="7.9375" y="21.59" smashed="yes" rot="MR90">
+<element name="R21" library="resistor" package="R0805" value="0.5R" x="7.9375" y="21.59" smashed="yes" rot="MR90">
 <attribute name="NAME" x="8.6995" y="18.4785" size="1.27" layer="26" rot="MR0"/>
 <attribute name="VALUE" x="5.6515" y="20.828" size="1.27" layer="28" rot="MR90"/>
@@
 <attribute name="VALUE" x="41.1988" y="36.9062" size="1.27" layer="27"/>
 </element>
-<element name="L1" library="keycopy" package="0207/2V" value="777uH" x="78.74" y="9.2075" smashed="yes" rot="R270">
-<attribute name="NAME" x="78.3717" y="12.1285" size="1.27" layer="25" ratio="10"/>
-<attribute name="VALUE" x="76.5048" y="9.2583" size="1.27" layer="27" ratio="10" rot="R270"/>
+<element name="L1" library="keycopy" package="0207/2V" value="777uH" x="78.4225" y="10.4775" smashed="yes" rot="R270">
+<attribute name="NAME" x="78.0542" y="13.3985" size="1.27" layer="25" ratio="10"/>
+<attribute name="VALUE" x="76.1873" y="10.5283" size="1.27" layer="27" ratio="10" rot="R270"/>
 </element>
 <element name="C8B" library="keycopy" package="C025-030X050" value="47n" x="32.385" y="3.4925" smashed="yes" rot="R270">
@@
 <attribute name="VALUE" x="45.72" y="3.81" size="1.27" layer="28" rot="MR90"/>
 </element>
-<element name="+3V" library="keycopy" package="1X02" value="" x="2.8575" y="27.94" smashed="yes" rot="R90">
-<attribute name="NAME" x="1.1938" y="25.4762" size="1.27" layer="25" ratio="10" rot="R270"/>
-<attribute name="VALUE" x="6.0325" y="25.4" size="1.27" layer="27" rot="R90"/>
+<element name="+3V" library="keycopy" package="1X02" value="" x="2.8575" y="27.6225" smashed="yes" rot="R90">
+<attribute name="NAME" x="1.1938" y="25.1587" size="1.27" layer="25" ratio="10" rot="R270"/>
+<attribute name="VALUE" x="6.0325" y="25.0825" size="1.27" layer="27" rot="R90"/>
 </element>
 <element name="J3" library="keycopy" package="R1206W" value="" x="23.495" y="28.2575" smashed="yes" rot="MR90">
@@
 <wire x1="15.6175" y1="21.59" x2="13.97" y2="21.59" width="0.6096" layer="16"/>
 <wire x1="6.985" y1="30.48" x2="8.5725" y2="33.9725" width="1.27" layer="16"/>
-<wire x1="6.985" y1="30.48" x2="2.8575" y2="29.21" width="1.27" layer="16"/>
+<wire x1="6.985" y1="30.48" x2="2.8575" y2="28.8925" width="1.27" layer="16"/>
 <wire x1="72.7075" y1="2.2225" x2="76.835" y2="6.0325" width="0.8128" layer="16"/>
 <wire x1="76.835" y1="6.0325" x2="80.9625" y2="6.0325" width="0.8128" layer="16"/>
@@
 <vertex x="86.36" y="6.985"/>
 <vertex x="86.36" y="11.7475"/>
-<vertex x="81.5975" y="11.7475"/>
-<vertex x="81.5975" y="13.335"/>
+<vertex x="82.8675" y="11.7475"/>
+<vertex x="82.8675" y="13.335"/>
 <vertex x="86.36" y="13.335"/>
 <vertex x="86.995" y="12.3825"/>
@@
 <contactref element="L1" pad="2"/>
 <contactref element="C1B*" pad="1"/>
-<wire x1="78.74" y1="7.9375" x2="77.47" y2="7.62" width="0.6096" layer="16"/>
-<wire x1="77.47" y1="7.62" x2="76.2" y2="7.62" width="0.6096" layer="16"/>
+<wire x1="78.4225" y1="9.2075" x2="76.2" y2="7.62" width="0.6096" layer="16"/>
 <wire x1="76.2" y1="7.62" x2="72.7075" y2="4.7625" width="0.6096" layer="16"/>
 <wire x1="72.7075" y1="4.7625" x2="69.5325" y2="4.7625" width="1.27" layer="16"/>
@@
 <wire x1="9.2075" y1="20.32" x2="7.9375" y2="20.74" width="0.4064" layer="16"/>
 <wire x1="13.0175" y1="26.9875" x2="11.7475" y2="28.2575" width="0.6096" layer="16"/>
-<wire x1="2.8575" y1="26.67" x2="6.985" y2="27.94" width="1.27" layer="16"/>
+<wire x1="2.8575" y1="26.3525" x2="6.985" y2="27.94" width="1.27" layer="16"/>
 <contactref element="VT2" pad="E"/>
 <wire x1="36.83" y1="17.78" x2="35.56" y2="17.78" width="0.4064" layer="16"/>
 <via x="35.56" y="17.78" extent="1-16" drill="0.8" diameter="2.3"/>
 <wire x1="35.56" y1="17.78" x2="16.51" y2="17.78" width="0.4064" layer="1"/>
-<wire x1="16.51" y1="17.78" x2="3.4925" y2="24.13" width="0.4064" layer="1"/>
-<via x="3.4925" y="24.13" extent="1-16" drill="0.8" diameter="2.3"/>
-<wire x1="3.4925" y1="24.13" x2="2.8575" y2="26.67" width="0.4064" layer="16"/>
+<wire x1="16.51" y1="17.78" x2="3.81" y2="23.8125" width="0.4064" layer="1"/>
+<via x="3.81" y="23.8125" extent="1-16" drill="0.8" diameter="2.3"/>
+<wire x1="3.81" y1="23.8125" x2="2.8575" y2="26.3525" width="0.4064" layer="16"/>
 <contactref element="R4*" pad="2"/>
 <wire x1="36.83" y1="17.78" x2="37.465" y2="19.52625" width="0.4064" layer="16"/>
@@
 <contactref element="L1" pad="1"/>
 <wire x1="74.6125" y1="13.97" x2="74.725" y2="16.8275" width="1.27" layer="16"/>
-<wire x1="74.6125" y1="13.97" x2="73.66" y2="9.525" width="1.27" layer="16"/>
-<wire x1="73.66" y1="9.525" x2="78.74" y2="10.4775" width="1.27" layer="16"/>
-<wire x1="78.74" y1="10.4775" x2="81.915" y2="10.2725" width="1.27" layer="16"/>
+<wire x1="74.6125" y1="13.97" x2="74.157159375" y2="11.845071875" width="1.27" layer="16"/>
+<wire x1="74.157159375" y1="11.845071875" x2="73.66" y2="9.525" width="1.27" layer="16"/>
+<wire x1="78.4225" y1="11.7475" x2="81.915" y2="10.2725" width="1.27" layer="16"/>
 <wire x1="81.915" y1="10.2725" x2="84.7725" y2="9.5225" width="1.27" layer="16"/>
+<wire x1="78.4225" y1="11.7475" x2="74.157159375" y2="11.845071875" width="1.016" layer="16"/>
 </signal>
 <signal name="N$1">

Commit message: 2016.07.05
Parts:
- L3: value 100uH -> 30uH
- R24: value 3k -> (3k&22k)
Connections:
- net N$5 renamed 1W_
Changed lines of the file:
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@@
 <setting verticaltext="up"/>
 </settings>
-<grid distance="12.5" unitdist="mil" unit="mil" style="lines" multiple="1" display="yes" altdistance="0.025" altunitdist="inch" altunit="inch"/>
+<grid distance="50" unitdist="mil" unit="mil" style="lines" multiple="1" display="yes" altdistance="0.025" altunitdist="inch" altunit="inch"/>
 <layers>
 <layer number="1" name="Top" color="4" fill="1" visible="yes" active="yes"/>
@@
 <attribute name="VALUE" x="13.462" y="15.494" size="1.27" layer="28" rot="MR0"/>
 </element>
-<element name="R24" library="resistor" package="R1206W" value="3k" x="9.525" y="16.1925" smashed="yes" rot="MR270">
+<element name="R24" library="resistor" package="R1206W" value="(3k&amp;22k)" x="9.525" y="16.1925" smashed="yes" rot="MR270">
 <attribute name="NAME" x="8.4455" y="10.7315" size="1.27" layer="26" rot="MR90"/>
 <attribute name="VALUE" x="11.938" y="17.8435" size="1.27" layer="28" rot="MR270"/>
@@
 <attribute name="VALUE" x="54.099165625" y="25.9108375" size="0.02" layer="28" rot="MR225"/>
 </element>
-<element name="L3" library="rcl" package="0207/12" value="100uH" x="26.9875" y="19.05" smashed="yes">
+<element name="L3" library="rcl" package="0207/12" value="30uH" x="26.9875" y="19.05" smashed="yes">
 <attribute name="NAME" x="25.7175" y="18.2245" size="1.27" layer="25" ratio="10"/>
 <attribute name="VALUE" x="24.7015" y="18.3642" size="1.27" layer="27" ratio="10"/>
@@
 <wire x1="13.106" y1="7.391" x2="27.6225" y2="7.391" width="0.3048" layer="16"/>
 <wire x1="27.6225" y1="7.391" x2="27.94" y2="7.7085" width="0.3048" layer="16"/>
-<wire x1="16.1671" y1="4.7625" x2="16.1671" y2="4.1021" width="0.254" layer="16"/>
-<wire x1="16.1671" y1="4.1021" x2="15.5575" y2="3.4925" width="0.254" layer="16"/>
-<wire x1="15.5575" y1="3.4925" x2="12.7" y2="3.4925" width="0.254" layer="16"/>
-<wire x1="12.7" y1="3.4925" x2="12.065" y2="4.1275" width="0.254" layer="16"/>
-<wire x1="12.065" y1="4.1275" x2="12.065" y2="5.715" width="0.254" layer="16"/>
+<wire x1="16.1671" y1="4.7625" x2="16.1671" y2="4.1021" width="0.3048" layer="16"/>
+<wire x1="16.1671" y1="4.1021" x2="15.5575" y2="3.4925" width="0.3048" layer="16"/>
+<wire x1="15.5575" y1="3.4925" x2="12.7" y2="3.4925" width="0.3048" layer="16"/>
+<wire x1="12.7" y1="3.4925" x2="12.065" y2="4.1275" width="0.3048" layer="16"/>
+<wire x1="12.065" y1="4.1275" x2="12.065" y2="5.715" width="0.3048" layer="16"/>
 </signal>
 <signal name="PGM">
@@
 <wire x1="79.375" y1="18.0975" x2="75.565" y2="19.3675" width="0.4064" layer="16"/>
 </signal>
-<signal name="N$5">
+<signal name="1W_">
 <contactref element="DD1" pad="6"/>
 <via x="30.1625" y="6.6675" extent="1-16" drill="0.8" diameter="2.3"/>
@@
 <wire x1="5.715" y1="7.62" x2="3.81" y2="7.62" width="0.4064" layer="16"/>
 <wire x1="20.22" y1="3.33375" x2="20.0025" y2="3.4925" width="0.4064" layer="16"/>
-<wire x1="20.0025" y1="3.4925" x2="18.7325" y2="2.8575" width="0.4064" layer="16"/>
-<wire x1="18.7325" y1="2.8575" x2="10.4775" y2="2.8575" width="0.4064" layer="16"/>
-<wire x1="10.4775" y1="2.8575" x2="5.715" y2="7.62" width="0.4064" layer="16"/>
+<wire x1="20.0025" y1="3.4925" x2="18.57375" y2="2.54" width="0.4064" layer="16"/>
+<wire x1="18.57375" y1="2.54" x2="10.4775" y2="2.54" width="0.4064" layer="16"/>
+<wire x1="10.4775" y1="2.54" x2="5.715" y2="7.62" width="0.4064" layer="16"/>
 </signal>
 <signal name="N$25">
