File: keycopy.sch (EAGLE design)
At the start: 85 parts

Commit message: b002
Parts:
- C1*: value 2n -> 2n2
- C1B*: value 2n -> (none)
- C8: value 150n -> 100n
- C8B: value 150n -> 47n
- DISP: value TUXGR_16X2_R21 -> QC1602A V2.0
- L1: value 820mkhn -> 777
- R: value 1k -> 10k
- TEST_PIN: value (none) -> +30V
Other:
- note added: "L1 ~ 743uH 150w 0.16mm d=19x19mm"

Commit message: v0.21
Parts:
- C14: value 47n -> 47m
- R3~: value 1k5 -> SMD
- VT1: device transistor-pnp:BD140 -> keycopy:BD140
- renumbered R3B to R3~
Connections:
- net V+: now also R4*.2, VT2.E
- net VCC/2: no longer R4*.2, VT2.E
Other:
- moved on the sheet: C3, R, R4*, R5, R7, R8, VD2, VT1, VT2

Commit message: v0.3
Parts:
- added R4: 1k, rcl:R-EU_R1206W
- L1: value 777 -> 777uH
- R4*: value 120 -> 20; device rcl:R-EU_R1206W -> rcl:R-EU_R0805
- VD2: value 3v9* -> 1v5*
- VT2: value КТ361 -> КТ361Б
Connections:
- new net N$38: R4*.1, R4.2
- net N$17: now also R4.1; no longer R4*.1
Other:
- note added: "VD2 T4148+LL4148+КД522Б 0,7v+0.7v+0.5v При точном резисторе 1.000k, пришлось подбирать диоды. Порог 2,5-2,6в, при этом на выходе около4,98в. Порог срабатывания увеличивается заменой импортных диодов на КД522 или увеличением сопротивления на 20ом, импортные слишком точные, придётся ставить второе"
- moved on the sheet: R4*, R5, R8, VD2, VT2

Commit message: v0.33
Parts:
- R21: value 1R -> 0.5R
Changed lines of the file:
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@@
 <part name="U$2" library="lib-user" deviceset="GND" device=""/>
 <part name="R22" library="resistor" deviceset="R-EU_" device="R0805" value="150"/>
-<part name="R21" library="resistor" deviceset="R-EU_" device="R0805" value="1R"/>
+<part name="R21" library="resistor" deviceset="R-EU_" device="R0805" value="0.5R"/>
 <part name="U$3" library="lib-user" deviceset="GND" device=""/>
 <part name="C10" library="keycopy" deviceset="CPOL-EU" device="E2.5-6" value="47n"/>
@@
 <pinref part="P+8" gate="VCC" pin="VCC"/>
 <pinref part="R" gate="G$1" pin="2"/>
-<wire x1="149.86" y1="139.7" x2="149.86" y2="137.16" width="0.1524" layer="91"/>
+<wire x1="149.86" y1="139.7" x2="149.86" y2="137.16" width="0.1524" layer="91" style="shortdash"/>
 </segment>
 </net>
@@
 <wire x1="149.86" y1="114.3" x2="139.7" y2="114.3" width="0.1524" layer="91"/>
 <pinref part="R" gate="G$1" pin="1"/>
-<wire x1="149.86" y1="127" x2="149.86" y2="114.3" width="0.1524" layer="91"/>
+<wire x1="149.86" y1="127" x2="149.86" y2="114.3" width="0.1524" layer="91" style="shortdash"/>
 <junction x="149.86" y="114.3"/>
 </segment>

Commit message: 2016.07.05
Parts:
- L3: value 100uH -> 30uH
- R24: value 3k -> (3k&22k)
Connections:
- net N$5 renamed 1W_
Other:
- note added: "+5.2v"
- moved on the sheet: DISP
Changed lines of the file:
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@@
 <part name="C10" library="keycopy" deviceset="CPOL-EU" device="E2.5-6" value="47n"/>
 <part name="R23" library="resistor" deviceset="R-EU_" device="R0805" value="1k"/>
-<part name="R24" library="resistor" deviceset="R-EU_" device="R1206W" value="3k"/>
+<part name="R24" library="resistor" deviceset="R-EU_" device="R1206W" value="(3k&amp;22k)"/>
 <part name="VD8" library="diode" deviceset="DIODE-" device="SMB" value="SS14"/>
 <part name="C15" library="resistor" deviceset="C-EU" device="C0805K" value="100n"/>
@@
 <part name="R3~" library="keycopy" deviceset="R-EU_" device="M0805" value="SMD"/>
 <part name="R" library="rcl" deviceset="R-EU_" device="R0805" value="10k"/>
-<part name="L3" library="rcl" deviceset="L-US" device="0207/12" value="100uH"/>
+<part name="L3" library="rcl" deviceset="L-US" device="0207/12" value="30uH"/>
 <part name="C13" library="rcl" deviceset="C-EU" device="C1210" value="22m"/>
 <part name="U$9" library="lib-user" deviceset="GND" device=""/>
@@
 импортные слишком точные, придётся ставить
 второе</text>
+<text x="314.96" y="163.83" size="1.778" layer="91">+5.2v</text>
 </plain>
 <instances>
@@
 <instance part="U$7" gate="G$1" x="241.3" y="116.84"/>
 <instance part="U$8" gate="G$1" x="241.3" y="134.62"/>
-<instance part="DISP" gate="G$1" x="238.76" y="45.72"/>
+<instance part="DISP" gate="G$1" x="316.23" y="91.44" rot="R270"/>
 <instance part="L1" gate="G$1" x="58.42" y="45.72" smashed="yes" rot="R90">
 <attribute name="NAME" x="60.96" y="52.07" size="1.778" layer="95" rot="R180"/>
@@
 </segment>
 </net>
-<net name="N$5" class="0">
+<net name="1W_" class="0">
 <segment>
 <pinref part="DD1" gate="G$1" pin="RB0/INT"/>
 <wire x1="38.1" y1="93.98" x2="33.02" y2="93.98" width="0.1524" layer="91"/>
-<label x="35.56" y="93.98" size="1.778" layer="95" rot="MR0"/>
+<label x="34.29" y="99.06" size="1.778" layer="95" rot="MR180"/>
 <wire x1="33.02" y1="93.98" x2="33.02" y2="144.78" width="0.1524" layer="91"/>
 <pinref part="J5" gate="G$1" pin="1"/>
